File: iov-rp2040.kicad_sch (KiCad schematic)
At the start: 43 parts, among them J1 USB_C_Receptacle_USB2.0, J2 SWD, J3 output header, Q1 BC847, SW1 CL-SB-13B-01T, SW2 BSL, SW3 RST, U1 TLV75518PDBV, U2 TLV75533PDBV, U3 AT25FF081A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

Commit message: revision b:
fixed flash footprint
changed ground pour to be cleaner
added name and revision text
Parts:
- U3: footprint Package_SO:SOIC-8_3.9x4.9mm_P1.27mm -> Package_SO:SOIC-8_5.275x5.275mm_P1.27mm
Changed lines of the file:
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@@
       (effects (font (size 1.27 1.27)) (justify left))
     )
-    (property "Footprint" "Package_SO:SOIC-8_3.9x4.9mm_P1.27mm" (id 2) (at 63.5 179.07 0)
+    (property "Footprint" "Package_SO:SOIC-8_5.275x5.275mm_P1.27mm" (id 2) (at 63.5 179.07 0)
       (effects (font (size 1.27 1.27)) hide)
     )
@@
     )
     (path "/b7b22185-0271-4de5-b512-c1d6d756b28e"
-      (reference "U3") (unit 1) (value "AT25FF081A") (footprint "Package_SO:SOIC-8_3.9x4.9mm_P1.27mm")
+      (reference "U3") (unit 1) (value "AT25FF081A") (footprint "Package_SO:SOIC-8_5.275x5.275mm_P1.27mm")
     )
     (path "/88204602-feae-4226-a97a-61e6ccfdf297"
